File: LinearSaturn.kicad_pcb (KiCad board)
At the start: 2 copper layers, 45.7 x 167.2 mm, 26 parts

Commit message: Signed-off-by: filip <bolo-poczta@outlook.com>
Parts:
- moved ? 15.8 mm to (142.6, 79.5)
- moved ? 15.8 mm to (142.6, 84.5)
- moved ? 15.8 mm to (142.6, 82.0)
Routing:
- net (no net): track 317.7 -> 296.6 mm
- net 5v: track 132.1 -> 113.1 mm
Other:
- board text added: "Linear Saturn PSU V3 VA-SD / VA-SG"
- board text removed: "Linear Saturn PSU V2.50 VA-SD / VA-SG"
Changed lines of the file:
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@@
 	)
 	(footprint ""
+		(locked yes)
 		(layer "F.Cu")
-		(at 146.024 69.144)
+		(at 142.564 84.54)
 		(property "Reference" ""
 			(at 0 0 0)
@@
 	)
 	(footprint ""
+		(locked yes)
 		(layer "F.Cu")
-		(at 146.024 66.604)
+		(at 142.564 82)
 		(property "Reference" ""
 			(at 0 0 0)
@@
 	)
 	(footprint ""
+		(locked yes)
 		(layer "F.Cu")
-		(at 146.024 64.064)
+		(at 142.564 79.46)
 		(property "Reference" ""
 			(at 0 0 0)
@@
 		)
 	)
-	(gr_text "Linear Saturn PSU V2.50\nVA-SD / VA-SG"
+	(gr_text "Linear Saturn PSU V3\nVA-SD / VA-SG"
 		(at 141.732 192.024 0)
 		(layer "F.SilkS")
@@
 	)
 	(gr_text "LM1084IT-5.0"
-		(at 137.5 61 0)
+		(at 133.5 76.5 0)
 		(layer "F.SilkS")
 		(effects
@@
 	)
 	(gr_text "-> Metal side\n<- Black side"
-		(at 136 75.5 0)
+		(at 132 91 0)
 		(layer "F.SilkS")
 		(effects
@@
 	)
 	(gr_text "9v IN"
-		(at 137 70 0)
+		(at 133 85.5 0)
 		(layer "F.SilkS")
 		(effects
@@
 	)
 	(gr_text "5v OUT"
-		(at 135.5 67.5 0)
+		(at 131.5 83 0)
 		(layer "F.SilkS")
 		(effects
@@
 	)
 	(gr_text "GND"
-		(at 139 65 0)
+		(at 135 80.5 0)
 		(layer "F.SilkS")
 		(effects
@@
 	)
 	(segment
-		(start 135.310379 143.256)
-		(end 136.358932 143.256)
-		(width 1)
-		(layer "B.Cu")
-		(net 0)
-	)
-	(segment
 		(start 135.128 143.256)
 		(end 135.310379 143.256)
@@
 	)
 	(segment
-		(start 141.986 75.514)
-		(end 146.024 71.476)
-		(width 2)
-		(layer "B.Cu")
-		(net 0)
-	)
-	(segment
-		(start 141.986 137.628932)
-		(end 141.986 75.514)
+		(start 130.81 61.761068)
+		(end 130.81 134.580932)
 		(width 2)
 		(layer "B.Cu")
@@
 	)
 	(segment
-		(start 138.43 143.256)
-		(end 140.521534 141.164466)
-		(width 0.25)
-		(layer "B.Cu")
-		(net 0)
-	)
-	(segment
-		(start 130.81 61.761068)
-		(end 130.81 134.580932)
+		(start 135.310379 143.256)
+		(end 142.564 136.002379)
 		(width 2)
 		(layer "B.Cu")
@@
 	)
 	(segment
-		(start 139.894466 141.791534)
-		(end 140.521534 141.164466)
-		(width 2)
-		(layer "B.Cu")
-		(net 0)
-	)
-	(segment
-		(start 146.024 71.476)
-		(end 146.024 69.144)
+		(start 142.564 136.002379)
+		(end 142.564 84.54)
 		(width 2)
 		(layer "B.Cu")
@@
 	)
 	(arc
-		(start 140.521534 141.164466)
-		(mid 141.605398 139.542349)
-		(end 141.986 137.628932)
-		(width 2)
-		(layer "B.Cu")
-		(net 0)
-	)
-	(arc
-		(start 136.358932 143.256)
-		(mid 138.272349 142.875398)
-		(end 139.894466 141.791534)
-		(width 2)
-		(layer "B.Cu")
-		(net 0)
-	)
-	(arc
 		(start 138.239311 166.433311)
 		(mid 136.071583 163.189077)
@@
 	)
 	(segment
+		(start 149.498 143.002)
+		(end 146.558 143.002)
+		(width 2)
+		(layer "B.Cu")
+		(net 3)
+	)
+	(segment
 		(start 144.272 144.654651)
 		(end 145.924651 143.002)
@@
 	)
 	(segment
-		(start 158.896 66.604)
-		(end 159.004 66.712)
+		(start 155.436 82)
+		(end 155.544 82.108)
 		(width 2)
+		(locked yes)
 		(layer "B.Cu")
 		(net 3)
@@
 	)
 	(segment
+		(start 155.544 82.108)
+		(end 155.5 82.152)
+		(width 2)
+		(layer "B.Cu")
+		(net 3)
+	)
+	(segment
 		(start 144.272 148.844)
 		(end 144.272 144.654651)
@@
 	)
 	(segment
-		(start 144.272 148.829436)
-		(end 144.272 144.654651)
-		(width 1.25)
+		(start 155.5 137)
+		(end 149.498 143.002)
+		(width 2)
 		(layer "B.Cu")
 		(net 3)
 	)
 	(segment
-		(start 149.019864 143.002)
-		(end 146.558 143.002)
+		(start 155.5 82.152)
+		(end 155.5 137)
 		(width 2)
 		(layer "B.Cu")
@@
 	)
 	(segment
-		(start 159.004 93.765068)
-		(end 159.004 135.088932)
-		(width 2)
+		(start 144.272 148.829436)
+		(end 144.272 144.654651)
+		(width 1.25)
 		(layer "B.Cu")
 		(net 3)
 	)
 	(segment
-		(start 151.732 151.036)
-		(end 146.464 151.036)
-		(width 1.25)
+		(start 155.5 137)
+		(end 154.75 137.75)
+		(width 2)
 		(layer "B.Cu")
 		(net 3)
 	)
 	(segment
-		(start 157.539534 138.624466)
-		(end 156.090932 140.073068)
-		(width 2)
+		(start 151.732 151.036)
+		(end 146.464 151.036)
+		(width 1.25)
 		(layer "B.Cu")
 		(net 3)
@@
 	)
 	(segment
-		(start 159.004 66.712)
-		(end 159.004 95.5)
-		(width 2)
-		(layer "B.Cu")
-		(net 3)
-	)
-	(segment
-		(start 146.024 66.604)
-		(end 158.896 66.604)
-		(width 2)
-		(layer "B.Cu")
-		(net 3)
-	)
-	(arc
-		(start 159.004 135.088932)
-		(mid 158.623398 137.002349)
-		(end 157.539534 138.624466)
-		(width 2)
-		(layer "B.Cu")
-		(net 3)
-	)
-	(arc
-		(start 156.090932 140.073068)
-		(mid 152.846698 142.240796)
-		(end 149.019864 143.002)
+		(start 142.564 82)
+		(end 155.436 82)
 		(width 2)
+		(locked yes)
 		(layer "B.Cu")
 		(net 3)
